File: Schematics/CameraBoard.kicad_pcb (KiCad board)
At the start: 4 copper layers, 50 x 100 mm, 73 parts, among them J1 Microsemi_FlashPro-JTAG-10, J2 USB_C_Receptacle, U1 STM32F405RGT6, U2 LDL1117-3.3, U3 TPS22917DBVR, U4 SN65HVD230, U5 TPS22917DBVR, U6 TPS22917DBVR, Y1 8mhz

Commit message: fixed schematic and named ready for bom to order
Parts:
- removed J2: USB_C_Receptacle, Connector_USB:USB_C_Receptacle_HRO_TYPE-C-31-M-12
- added G***: LOGO, LOGO, F.Cu at (78.8, 51.6)
- added J3: USB_C_Receptacle_USB2.0_16P, Connector_USB:USB_C_Receptacle_HRO_TYPE-C-31-M-12, F.Cu at (75.7, 67.7)
- C16: value 1u -> 100nf
- C17: value 4.7u -> 10u
- moved C15 0.37 mm to (99.1, 66.6)
- moved C14 0.37 mm to (103.8, 68.3)
- moved Y1 0.37 mm to (102.6, 65.2)
- moved BootSwitch1 0.25 mm to (116.7, 83.5)
Connections:
- U1 pad 33: /Can_transceiver/CAN_RX_2 -> /Can_transceiver/CAN_TX_2
- U1 pad 34: /Can_transceiver/CAN_TX_2 -> /Can_transceiver/CAN_RX_2
Routing:
- net /MCU/OSC OUT: track 10.1 -> 6.40 mm
- net GND: track 109.9 -> 113.4 mm, vias 42 -> 54
- net /Camera_right/PWN_EN: track 58.5 -> 56.5 mm
- net /MCU/OSC IN: track 9.72 -> 7.94 mm
- net /Can_transceiver/CAN_RX_2: track 28.2 -> 26.9 mm
- net /Can_transceiver/CANL: track 32.6 -> 31.4 mm
- net /MCU/SWCLK: track 64.8 -> 66.0 mm, vias 2 -> 1
- net /Camera_left/PWN_EN: track 41.1 -> 39.9 mm
- net +3.3V: track 62.3 -> 61.1 mm
- net /Can_transceiver/CAN_TX_2: track 31.6 -> 30.8 mm
- net /MCU/SWDIO: track 55.5 -> 54.9 mm
- added copper zone on F.Cu, net +3.3V
- removed copper zone on F.Cu, net (none)
Other:
- board text added: "Can"
- board text added: "Raven"
- board text added: "by Reetabass"
- board text removed: "Can In"
- board text removed: "Can Out"
- board text removed: "More Core Division"
