File: Schematics/CameraBoard.kicad_pcb (KiCad board)
At the start: 4 copper layers, 50 x 100 mm, 73 parts, among them J1 Microsemi_FlashPro-JTAG-10, J3 USB_C_Receptacle_USB2.0_16P, U1 STM32F405RGT6, U2 LDL1117-3.3, U3 TPS22917DBVR, U4 SN65HVD230, U5 TPS22917DBVR, U6 TPS22917DBVR, Y1 8mhz

Commit message: updating schematic for final order
Parts:
- moved G*** 6.36 mm to (83.7, 51.4)
