File: Schematics/power.kicad_sch (KiCad schematic)
At the start: 10 parts, among them U2 LDL1117-3.3

Commit message: output files completed quote obtained
Parts:
- C16: LCSC (none) -> C49678
- C17: LCSC (none) -> C98192
- D2, D3: LCSC (none) -> C113936
- U2: LCSC (none) -> C435835
Changed lines of the file:
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@@
 			)
 		)
-		(property "LCSC" ""
+		(property "LCSC" "C113936"
 			(at 74.93 102.87 90)
 			(effects
@@
 			)
 		)
-		(property "LCSC" ""
+		(property "LCSC" "C435835"
 			(at 155.956 121.412 0)
 			(effects
@@
 			)
 		)
+		(property "LCSC" "C98192"
+			(at 172.72 113.03 0)
+			(effects
+				(font
+					(size 1.27 1.27)
+				)
+				(hide yes)
+			)
+		)
 		(pin "2"
 		)
@@
 			)
 		)
-		(property "LCSC" ""
+		(property "LCSC" "C113936"
 			(at 92.71 102.87 90)
 			(effects
@@
 			(at 118.11 113.03 0)
 			(effects
+				(font
+					(size 1.27 1.27)
+				)
+				(hide yes)
+			)
+		)
+		(property "LCSC" "C49678"
+			(at 118.11 113.03 0)
+			(effects

Commit message: final output files
Parts:
- C17: LCSC C98192 -> C2932476
Changed lines of the file:
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@@
 			)
 		)
-		(property "LCSC" "C98192"
+		(property "LCSC" "C2932476"
 			(at 172.72 113.03 0)
 			(effects

Commit message: fixed can tranciver issues and updated to KiCad 10.0
Parts:
- J_BUCK_IN_A1, J_BUCK_IN_B1, J_BUCK_OUT_A1, J_BUCK_OUT_B1: value ~ -> (none)
