File: Schematics/power.kicad_sch (KiCad schematic)
At the start: 10 parts, among them U2 LDL1117-3.3

Commit message: updated stlink connector
Parts:
- C17: LCSC C2932476 -> C15850
Changed lines of the file:
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@@
 			)
 		)
-		(property "Description" "Generic connector, single row, 01x02, script generated (kicad-library-utils/schlib/autogen/connector/)"
+		(property "Description" ""
 			(at 156.21 64.77 0)
 			(hide yes)
@@
 			)
 		)
-		(property "Description" "Schottky diode"
-			(at 74.93 102.87 0)
+		(property "Description" ""
+			(at 74.93 102.87 90)
 			(hide yes)
 			(show_name no)
@@
 			)
 		)
-		(property "Description" "Generic connector, single row, 01x02, script generated (kicad-library-utils/schlib/autogen/connector/)"
+		(property "Description" ""
 			(at 139.7 62.23 0)
 			(hide yes)
@@
 			)
 		)
-		(property "Description" "Generic connector, single row, 01x02, script generated (kicad-library-utils/schlib/autogen/connector/)"
+		(property "Description" ""
 			(at 156.21 58.42 0)
 			(hide yes)
@@
 			)
 		)
-		(property "Description" "Unpolarized capacitor"
+		(property "Description" ""
 			(at 172.72 113.03 0)
 			(hide yes)
@@
 			)
 		)
-		(property "LCSC" "C2932476"
+		(property "LCSC" "C15850"
 			(at 172.72 113.03 0)
 			(hide yes)
@@
 			)
 		)
-		(property "Description" "Schottky diode"
-			(at 92.71 102.87 0)
+		(property "Description" ""
+			(at 92.71 102.87 90)
 			(hide yes)
 			(show_name no)
@@
 			)
 		)
-		(property "Description" "Generic connector, single row, 01x02, script generated (kicad-library-utils/schlib/autogen/connector/)"
+		(property "Description" ""
 			(at 104.14 60.96 0)
 			(hide yes)
@@
 			)
 		)
-		(property "Description" "Unpolarized capacitor"
+		(property "Description" ""
 			(at 118.11 113.03 0)
 			(hide yes)
@@
 			)
 		)
-		(property "Description" "Generic connector, single row, 01x02, script generated (kicad-library-utils/schlib/autogen/connector/)"
+		(property "Description" ""
 			(at 139.7 55.88 0)
 			(hide yes)
