File: Schematics/usb_type_c_sch.kicad_sch (KiCad schematic)
At the start: 4 parts, among them J3 USB_C_Receptacle_USB2.0_16P

Commit message: output files completed quote obtained
Parts:
- J3: LCSC (none) -> C165948
Changed lines of the file:
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@@
+			)
+		)
+		(property "LCSC" "C165948"
+			(at 125.73 82.55 0)
+			(effects
+				(font
+					(size 1.27 1.27)
+				)
+				(hide yes)
 			)
 		)

Commit message: fixed can tranciver issues and updated to KiCad 10.0
Parts:
- D4: DESCRIPTION Semtech SRV05-4.TCT, Uni-Directional TVS Diode Array, 300W,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 -> (none)
