File: Schematics/MCU.kicad_sch (KiCad schematic)
At the start: 27 parts, among them J1 Microsemi_FlashPro-JTAG-10, U1 STM32F405RGT6, Y1 8mhz

Commit message: updating schematic for final order
Parts:
- R1: value 10kr -> 10k
- R2: value 100kr -> 10k; LCSC C149504 -> C84376
Changed lines of the file:
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@@
 			)
 		)
-		(property "Value" "10kr"
+		(property "Value" "10k"
 			(at 38.1 49.53 90)
 			(show_name no)
@@
 			)
 		)
-		(property "Value" "100kr"
+		(property "Value" "10k"
 			(at 38.1 105.41 90)
 			(show_name no)
@@
 			)
 		)
-		(property "LCSC" "C149504"
+		(property "LCSC" "C84376"
 			(at 38.1 109.22 90)
 			(hide yes)
