File: Schematics/Camera.kicad_sch (KiCad schematic)
At the start: 7 parts, among them U3 TPS22917DBVR

Commit message: updated stlink connector
Parts:
- R5: LCSC C96346 -> C149504
Changed lines of the file:
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@@
 			)
 		)
-		(property "Description" "Unpolarized capacitor"
+		(property "Description" ""
 			(at 137.16 93.98 0)
 			(hide yes)
@@
 			)
 		)
-		(property "Description" "Unpolarized capacitor"
+		(property "Description" ""
 			(at 58.42 86.36 0)
 			(hide yes)
@@
 			)
 		)
-		(property "Description" "Unpolarized capacitor"
+		(property "Description" ""
 			(at 114.3 93.98 0)
 			(hide yes)
@@
 			)
 		)
-		(property "Description" "Resistor"
+		(property "Description" ""
 			(at 58.42 99.06 0)
 			(hide yes)
@@
 			)
 		)
-		(property "LCSC" "C96346"
+		(property "LCSC" "C149504"
 			(at 58.42 99.06 0)
 			(hide yes)
@@
 			)
 		)
-		(property "Description" "Generic connector, single row, 01x03, script generated (kicad-library-utils/schlib/autogen/connector/)"
+		(property "Description" ""
 			(at 219.71 93.98 0)
 			(hide yes)
@@
 			)
 		)
-		(property "Description" "Unpolarized capacitor"
+		(property "Description" ""
 			(at 127 93.98 0)
 			(hide yes)
