File: Schematics/Can_transceiver.kicad_sch (KiCad schematic)
At the start: 6 parts, among them U4 SN65HVD230

Commit message: fixed can tranciver issues and updated to KiCad 10.0
Parts:
- U4: LCSC C1543812 -> C12084

Commit message: updated stlink connector
Parts:
- R6: LCSC C114245 -> C17437
Changed lines of the file:
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@@
 			)
 		)
-		(property "Description" "Solder Jumper, 2-pole, open"
+		(property "Description" ""
 			(at 137.16 113.03 0)
 			(hide yes)
@@
 			)
 		)
-		(property "Description" "Generic connector, single row, 01x02, script generated (kicad-library-utils/schlib/autogen/connector/)"
+		(property "Description" ""
 			(at 173.99 104.14 0)
 			(hide yes)
@@
 			)
 		)
-		(property "Description" "Unpolarized capacitor"
+		(property "Description" ""
 			(at 77.47 109.22 0)
 			(hide yes)
@@
 			)
 		)
-		(property "Description" "CAN Bus Transceivers, 3.3V, 1Mbps, Low-Power capabilities, SOIC-8"
+		(property "Description" ""
 			(at 116.84 107.95 0)
 			(hide yes)
@@
 			)
 		)
-		(property "Description" "Resistor"
+		(property "Description" ""
 			(at 132.08 109.22 0)
 			(hide yes)
@@
 			)
 		)
-		(property "LCSC" "C114245"
+		(property "LCSC" " C17437"
 			(at 132.08 109.22 0)
 			(hide yes)
@@
 			)
 		)
-		(property "Description" "Generic connector, single row, 01x02, script generated (kicad-library-utils/schlib/autogen/connector/)"
+		(property "Description" ""
 			(at 173.99 113.03 0)
 			(hide yes)
